Commit message: Implemented dynamic-goal Q-learning with systematic training and BFS validation

File: ros2_ws/src/robot_description/urdf/robot.urdf.xacro (robot description, xacro)
@@ -1,7 +1,20 @@
 <?xml version="1.0"?>
-<robot name="rl_robot" xmlns:xacro="http://www.ros.org/wiki/xacro">
-  <!-- ================= BASE ================= -->
+<robot name="rl_robot"
+       xmlns:xacro="http://www.ros.org/wiki/xacro">
+  <!-- ===================================================== -->
+  <!-- BASE FOOTPRINT                                        -->
+  <!-- ===================================================== -->
+  <link name="base_footprint"/>
+  <joint name="base_footprint_joint" type="fixed">
+    <parent link="base_footprint"/>
+    <child link="base_link"/>
+    <origin xyz="0 0 0.125" rpy="0 0 0"/>
+  </joint>
+  <!-- ===================================================== -->
+  <!-- BASE LINK                                             -->
+  <!-- ===================================================== -->
   <link name="base_link">
     <visual>
+      <origin xyz="0 0 0" rpy="0 0 0"/>
       <geometry>
         <box size="0.40 0.30 0.15"/>
@@ -12,4 +25,5 @@
     </visual>
     <collision>
+      <origin xyz="0 0 0" rpy="0 0 0"/>
       <geometry>
         <box size="0.40 0.30 0.15"/>
@@ -17,30 +31,307 @@
     </collision>
     <inertial>
-      <origin xyz="0 0 0"/>
+      <origin xyz="0 0 0" rpy="0 0 0"/>
       <mass value="5.0"/>
       <inertia
-        ixx="0.05"
-        ixy="0.0"
-        ixz="0.0"
-        iyy="0.08"
-        iyz="0.0"
-        izz="0.10"/>
-    </inertial>
-  </link>
-  <!-- ================= LIDAR ================= -->
+        ixx="0.046875"
+        ixy="0.0"
+        ixz="0.0"
+        iyy="0.076042"
+        iyz="0.0"
+        izz="0.104167"/>
+    </inertial>
+  </link>
+  <!-- ===================================================== -->
+  <!-- LEFT WHEEL                                            -->
+  <!-- ===================================================== -->
+  <link name="left_wheel_link">
+    <visual>
+      <origin xyz="0 0 0" rpy="1.5708 0 0"/>
+      <geometry>
+        <cylinder
+          radius="0.075"
+          length="0.04"/>
+      </geometry>
+      <material name="black">
+        <color rgba="0.05 0.05 0.05 1"/>
+      </material>
+    </visual>
+    <collision>
+      <origin xyz="0 0 0" rpy="1.5708 0 0"/>
+      <geometry>
+        <cylinder
+          radius="0.075"
+          length="0.04"/>
+      </geometry>
+    </collision>
+    <inertial>
+      <origin xyz="0 0 0" rpy="0 0 0"/>
+      <mass value="0.5"/>
+      <inertia
+        ixx="0.001"
+        ixy="0.0"
+        ixz="0.0"
+        iyy="0.001"
+        iyz="0.0"
+        izz="0.001"/>
+    </inertial>
+  </link>
+  <joint name="left_wheel_joint" type="continuous">
+    <parent link="base_link"/>
+    <child link="left_wheel_link"/>
+    <origin
+      xyz="0 0.17 -0.05"
+      rpy="0 0 0"/>
+    <axis xyz="0 1 0"/>
+    <dynamics
+      damping="0.1"
+      friction="0.1"/>
+  </joint>
+  <!-- ===================================================== -->
+  <!-- RIGHT WHEEL                                           -->
+  <!-- ===================================================== -->
+  <link name="right_wheel_link">
+    <visual>
+      <origin xyz="0 0 0" rpy="1.5708 0 0"/>
+      <geometry>
+        <cylinder
+          radius="0.075"
+          length="0.04"/>
+      </geometry>
+      <material name="black">
+        <color rgba="0.05 0.05 0.05 1"/>
+      </material>
+    </visual>
+    <collision>
+      <origin xyz="0 0 0" rpy="1.5708 0 0"/>
+      <geometry>
+        <cylinder
+          radius="0.075"
+          length="0.04"/>
+      </geometry>
+    </collision>
+    <inertial>
+      <origin xyz="0 0 0" rpy="0 0 0"/>
+      <mass value="0.5"/>
+      <inertia
+        ixx="0.001"
+        ixy="0.0"
+        ixz="0.0"
+        iyy="0.001"
+        iyz="0.0"
+        izz="0.001"/>
+    </inertial>
+  </link>
+  <joint name="right_wheel_joint" type="continuous">
+    <parent link="base_link"/>
+    <child link="right_wheel_link"/>
+    <origin
+      xyz="0 -0.17 -0.05"
+      rpy="0 0 0"/>
+    <axis xyz="0 1 0"/>
+    <dynamics
+      damping="0.0"
+      friction="0.0"/>
+  </joint>
+  <!-- ===================================================== -->
+  <!-- REAR CASTER                                           -->
+  <!-- ===================================================== -->
+  <link name="caster_link">
+    <visual>
+      <origin xyz="0 0 0" rpy="0 0 0"/>
+      <geometry>
+        <sphere radius="0.04"/>
+      </geometry>
+      <material name="caster_gray">
+        <color rgba="0.3 0.3 0.3 1"/>
+      </material>
+    </visual>
+    <collision>
+      <origin xyz="0 0 0" rpy="0 0 0"/>
+      <geometry>
+        <sphere radius="0.04"/>
+      </geometry>
+    </collision>
+    <inertial>
+      <origin xyz="0 0 0" rpy="0 0 0"/>
+      <mass value="0.1"/>
+      <inertia
+        ixx="0.0001"
+        ixy="0.0"
+        ixz="0.0"
+        iyy="0.0001"
+        iyz="0.0"
+        izz="0.0001"/>
+    </inertial>
+  </link>
+  <joint name="caster_joint" type="fixed">
+    <parent link="base_link"/>
+    <child link="caster_link"/>
+    <!-- Fixed caster z-offset from -0.09 to -0.05 to prevent ground penetration -->
+    <origin
+      xyz="-0.14 0 -0.05"
+      rpy="0 0 0"/>
+  </joint>
+  <!-- ===================================================== -->
+  <!-- LIDAR                                                 -->
+  <!-- ===================================================== -->
   <link name="lidar_link">
     <visual>
-      <geometry>
-        <cylinder radius="0.04" length="0.03"/>
-      </geometry>
-      <material name="black">
+      <origin xyz="0 0 0" rpy="0 0 0"/>
+      <geometry>
+        <cylinder
+          radius="0.04"
+          length="0.03"/>
+      </geometry>
+      <material name="lidar_black">
         <color rgba="0 0 0 1"/>
       </material>
     </visual>
+    <inertial>
+      <origin xyz="0 0 0" rpy="0 0 0"/>
+      <mass value="0.05"/>
+      <inertia
+        ixx="0.0001"
+        ixy="0.0"
+        ixz="0.0"
+        iyy="0.0001"
+        iyz="0.0"
+        izz="0.0001"/>
+    </inertial>
   </link>
   <joint name="lidar_joint" type="fixed">
     <parent link="base_link"/>
     <child link="lidar_link"/>
-    <origin xyz="0 0 0.10" rpy="0 0 0"/>
-  </joint>
+    <origin
+      xyz="0 0 0.10"
+      rpy="0 0 0"/>
+  </joint>
+  <!-- ===================================================== -->
+  <!-- LIDAR GAZEBO SENSOR                                   -->
+  <!-- ===================================================== -->
+  <gazebo reference="lidar_link">
+    <sensor
+      name="lidar_sensor"
+      type="ray">
+      <pose>0 0 0 0 0 0</pose>
+      <visualize>true</visualize>
+      <update_rate>10</update_rate>
+      <always_on>true</always_on>
+      <ray>
+        <scan>
+          <horizontal>
+            <samples>360</samples>
+            <resolution>1</resolution>
+            <min_angle>-3.14159</min_angle>
+            <max_angle>3.14159</max_angle>
+          </horizontal>
+        </scan>
+        <range>
+          <min>0.12</min>
+          <max>10.0</max>
+          <resolution>0.01</resolution>
+        </range>
+      </ray>
+      <plugin
+        name="gazebo_ros_lidar"
+        filename="libgazebo_ros_ray_sensor.so">
+        <ros>
+          <namespace>/</namespace>
+          <remapping>~/out:=scan</remapping>
+        </ros>
+        <output_type>
+          sensor_msgs/LaserScan
+        </output_type>
+        <frame_name>
+          lidar_link
+        </frame_name>
+      </plugin>
+    </sensor>
+  </gazebo>
+  <!-- ===================================================== -->
+  <!-- GAZEBO MATERIALS                                      -->
+  <!-- ===================================================== -->
+  <gazebo reference="base_link">
+    <material>
+      Gazebo/Blue
+    </material>
+  </gazebo>
+  <gazebo reference="left_wheel_link">
+    <material>
+      Gazebo/Black
+    </material>
+    <mu1>1.0</mu1>
+    <mu2>1.0</mu2>
+    <kp>1000000.0</kp>
+    <kd>1.0</kd>
+  </gazebo>
+  <gazebo reference="right_wheel_link">
+    <material>
+      Gazebo/Black
+    </material>
+    <mu1>1.0</mu1>
+    <mu2>1.0</mu2>
+    <kp>1000000.0</kp>
+    <kd>1.0</kd>
+  </gazebo>
+  <!-- ===================================================== -->
+  <!-- LOW FRICTION CASTER                                   -->
+  <!-- ===================================================== -->
+  <gazebo reference="caster_link">
+    <mu1>0.01</mu1>
+    <mu2>0.01</mu2>
+    <kp>1000000.0</kp>
+    <kd>1.0</kd>
+  </gazebo>
+  <!-- ===================================================== -->
+  <!-- DIFFERENTIAL DRIVE PLUGIN                             -->
+  <!-- ===================================================== -->
+  <gazebo>
+    <plugin
+      name="diff_drive"
+      filename="libgazebo_ros_diff_drive.so">
+      <ros>
+        <namespace>/</namespace>
+      </ros>
+      <left_joint>
+        left_wheel_joint
+      </left_joint>
+      <right_joint>
+        right_wheel_joint
+      </right_joint>
+      <wheel_separation>
+        0.34
+      </wheel_separation>
+      <wheel_diameter>
+        0.15
+      </wheel_diameter>
+      <max_wheel_torque>
+        20.0
+      </max_wheel_torque>
+      <max_wheel_acceleration>
+        5.0
+      </max_wheel_acceleration>
+      <command_topic>
+        cmd_vel
+      </command_topic>
+      <odometry_topic>
+        odom
+      </odometry_topic>
+      <odometry_frame>
+        odom
+      </odometry_frame>
+      <robot_base_frame>
+        base_footprint
+      </robot_base_frame>
+      <publish_odom>
+        true
+      </publish_odom>
+      <publish_odom_tf>
+        true
+      </publish_odom_tf>
+      <publish_wheel_tf>
+        true
+      </publish_wheel_tf>
+    </plugin>
+  </gazebo>
 </robot>
