Commit message: Update RL Ackermann simulation and training

File: ros2_ws/src/robot_description/urdf/robot.urdf.xacro (robot description, xacro)
@@ -2,4 +2,28 @@
 <robot name="rl_robot"
        xmlns:xacro="http://www.ros.org/wiki/xacro">
+  <!-- =====================================================
+       Geometry updated to official Hiwonder chassis values
+       plus firmware constants:
+         - chassis plate: 270 x 120.5 x 2 mm (modeled as a
+           270 x 120.5 x 50 mm box - height is still a
+           modeling approximation, Hiwonder doesn't publish
+           assembled chassis height)
+         - wheel diameter: 60 mm (radius 0.03 m) - official
+         - wheelbase: 0.18 m (Hiwonder MINACKER_WHEELBASE)
+         - track width: 0.17 m (Hiwonder MINACKER_SHAFT_LENGTH)
+         - front axle x = +0.09, rear axle x = -0.09
+         - left wheel y = +0.085, right wheel y = -0.085
+         - ground clearance under chassis = 0.02 m (estimate)
+       STILL UNKNOWN / PLACEHOLDER:
+         - base_link mass (kept at 5.0 kg - bare plate is only
+           ~126 g, but full robot with motors/servo/battery/
+           compute/lidar will weigh more; update once assembled
+           and weighed)
+         - wheel / knuckle masses (placeholders)
+         - steering angle limit (0.6 rad / ~34 deg is an estimate,
+           actual range depends on the LD-1501MG + linkage geometry)
+         - lidar mounting height (unchanged until RPLIDAR A1 is
+           physically installed)
+  ===================================================== -->
   <!-- ===================================================== -->
   <!-- BASE FOOTPRINT                                        -->
@@ -9,5 +33,6 @@
     <parent link="base_footprint"/>
     <child link="base_link"/>
-    <origin xyz="0 0 0.125" rpy="0 0 0"/>
+    <!-- ground clearance (0.02) + half chassis height (0.025) -->
+    <origin xyz="0 0 0.05" rpy="0 0 0"/>
   </joint>
   <!-- ===================================================== -->
@@ -18,5 +43,5 @@
       <origin xyz="0 0 0" rpy="0 0 0"/>
       <geometry>
-        <box size="0.40 0.30 0.15"/>
+        <box size="0.270 0.1205 0.050"/>
       </geometry>
       <material name="blue">
@@ -27,29 +52,77 @@
       <origin xyz="0 0 0" rpy="0 0 0"/>
       <geometry>
-        <box size="0.40 0.30 0.15"/>
+        <box size="0.270 0.1205 0.050"/>
       </geometry>
     </collision>
     <inertial>
       <origin xyz="0 0 0" rpy="0 0 0"/>
-      <mass value="5.0"/>
+      <!-- mass is still a placeholder - bare Hiwonder plate is ~126 g,
+           but full robot (motors/servo/battery/compute/lidar) will be
+           heavier. Update once the robot is assembled and weighed. -->
+      <mass value="2.5"/>
       <inertia
-        ixx="0.046875"
+        ixx="0.003546"
         ixy="0.0"
         ixz="0.0"
-        iyy="0.076042"
+        iyy="0.015708"
         iyz="0.0"
-        izz="0.104167"/>
-    </inertial>
-  </link>
-  <!-- ===================================================== -->
-  <!-- LEFT WHEEL                                            -->
-  <!-- ===================================================== -->
-  <link name="left_wheel_link">
-    <visual>
-      <origin xyz="0 0 0" rpy="1.5708 0 0"/>
-      <geometry>
-        <cylinder
-          radius="0.075"
-          length="0.04"/>
+        izz="0.018213"/>
+    </inertial>
+  </link>
+  <!-- ===================================================== -->
+  <!-- STEERING LINK (virtual)                                -->
+  <!-- Required only because libgazebo_ros_ackermann_drive.so -->
+  <!-- looks for a steering_wheel_joint parameter. This does   -->
+  <!-- not drive anything physically - the real steering      -->
+  <!-- happens through front_left/right_steering_joint below.  -->
+  <!-- ===================================================== -->
+  <link name="steering_link">
+    <inertial>
+      <origin xyz="0 0 0" rpy="0 0 0"/>
+      <mass value="0.001"/>
+      <inertia
+        ixx="0.000001"
+        ixy="0.0"
+        ixz="0.0"
+        iyy="0.000001"
+        iyz="0.0"
+        izz="0.000001"/>
+    </inertial>
+  </link>
+  <joint name="steering_joint" type="revolute">
+    <parent link="base_link"/>
+    <child link="steering_link"/>
+    <origin xyz="0 0 0.05" rpy="0 0 0"/>
+    <axis xyz="0 0 1"/>
+    <limit
+      lower="-7.85"
+      upper="7.85"
+      effort="10"
+      velocity="10"/>
+  </joint>
+  <!-- ===================================================== -->
+  <!-- FRONT LEFT STEERING KNUCKLE + WHEEL                    -->
+  <!-- ===================================================== -->
+  <link name="front_left_steering_link">
+    <inertial>
+      <origin xyz="0 0 0" rpy="0 0 0"/>
+      <mass value="0.05"/>
+      <inertia ixx="0.00001" ixy="0.0" ixz="0.0"
+                iyy="0.00001" iyz="0.0" izz="0.00001"/>
+    </inertial>
+  </link>
+  <joint name="front_left_steering_joint" type="revolute">
+    <parent link="base_link"/>
+    <child link="front_left_steering_link"/>
+    <origin xyz="0.09 0.085 -0.03" rpy="0 0 0"/>
+    <axis xyz="0 0 1"/>
+    <limit lower="-0.6" upper="0.6" effort="10" velocity="5"/>
+    <dynamics damping="0.05" friction="0.05"/>
+  </joint>
+  <link name="front_left_wheel_link">
+    <visual>
+      <origin xyz="0 0 0" rpy="1.5708 0 0"/>
+      <geometry>
+        <cylinder radius="0.03" length="0.02"/>
       </geometry>
       <material name="black">
@@ -60,42 +133,45 @@
       <origin xyz="0 0 0" rpy="1.5708 0 0"/>
       <geometry>
-        <cylinder
-          radius="0.075"
-          length="0.04"/>
+        <cylinder radius="0.03" length="0.02"/>
       </geometry>
     </collision>
     <inertial>
       <origin xyz="0 0 0" rpy="0 0 0"/>
-      <mass value="0.5"/>
-      <inertia
-        ixx="0.001"
-        ixy="0.0"
-        ixz="0.0"
-        iyy="0.001"
-        iyz="0.0"
-        izz="0.001"/>
-    </inertial>
-  </link>
-  <joint name="left_wheel_joint" type="continuous">
-    <parent link="base_link"/>
-    <child link="left_wheel_link"/>
-    <origin
-      xyz="0 0.17 -0.05"
-      rpy="0 0 0"/>
+      <mass value="0.15"/>
+      <inertia ixx="0.0001" ixy="0.0" ixz="0.0"
+                iyy="0.0001" iyz="0.0" izz="0.0001"/>
+    </inertial>
+  </link>
+  <joint name="front_left_wheel_joint" type="continuous">
+    <parent link="front_left_steering_link"/>
+    <child link="front_left_wheel_link"/>
+    <origin xyz="0 0 0" rpy="0 0 0"/>
     <axis xyz="0 1 0"/>
-    <dynamics
-      damping="0.1"
-      friction="0.1"/>
-  </joint>
-  <!-- ===================================================== -->
-  <!-- RIGHT WHEEL                                           -->
-  <!-- ===================================================== -->
-  <link name="right_wheel_link">
-    <visual>
-      <origin xyz="0 0 0" rpy="1.5708 0 0"/>
-      <geometry>
-        <cylinder
-          radius="0.075"
-          length="0.04"/>
+    <dynamics damping="0.1" friction="0.1"/>
+  </joint>
+  <!-- ===================================================== -->
+  <!-- FRONT RIGHT STEERING KNUCKLE + WHEEL                   -->
+  <!-- ===================================================== -->
+  <link name="front_right_steering_link">
+    <inertial>
+      <origin xyz="0 0 0" rpy="0 0 0"/>
+      <mass value="0.05"/>
+      <inertia ixx="0.00001" ixy="0.0" ixz="0.0"
+                iyy="0.00001" iyz="0.0" izz="0.00001"/>
+    </inertial>
+  </link>
+  <joint name="front_right_steering_joint" type="revolute">
+    <parent link="base_link"/>
+    <child link="front_right_steering_link"/>
+    <origin xyz="0.09 -0.085 -0.03" rpy="0 0 0"/>
+    <axis xyz="0 0 1"/>
+    <limit lower="-0.6" upper="0.6" effort="10" velocity="5"/>
+    <dynamics damping="0.05" friction="0.05"/>
+  </joint>
+  <link name="front_right_wheel_link">
+    <visual>
+      <origin xyz="0 0 0" rpy="1.5708 0 0"/>
+      <geometry>
+        <cylinder radius="0.03" length="0.02"/>
       </geometry>
       <material name="black">
@@ -106,73 +182,89 @@
       <origin xyz="0 0 0" rpy="1.5708 0 0"/>
       <geometry>
-        <cylinder
-          radius="0.075"
-          length="0.04"/>
+        <cylinder radius="0.03" length="0.02"/>
       </geometry>
     </collision>
     <inertial>
       <origin xyz="0 0 0" rpy="0 0 0"/>
-      <mass value="0.5"/>
-      <inertia
-        ixx="0.001"
-        ixy="0.0"
-        ixz="0.0"
-        iyy="0.001"
-        iyz="0.0"
-        izz="0.001"/>
-    </inertial>
-  </link>
-  <joint name="right_wheel_joint" type="continuous">
-    <parent link="base_link"/>
-    <child link="right_wheel_link"/>
-    <origin
-      xyz="0 -0.17 -0.05"
-      rpy="0 0 0"/>
+      <mass value="0.15"/>
+      <inertia ixx="0.0001" ixy="0.0" ixz="0.0"
+                iyy="0.0001" iyz="0.0" izz="0.0001"/>
+    </inertial>
+  </link>
+  <joint name="front_right_wheel_joint" type="continuous">
+    <parent link="front_right_steering_link"/>
+    <child link="front_right_wheel_link"/>
+    <origin xyz="0 0 0" rpy="0 0 0"/>
     <axis xyz="0 1 0"/>
-    <dynamics
-      damping="0.0"
-      friction="0.0"/>
-  </joint>
-  <!-- ===================================================== -->
-  <!-- REAR CASTER                                           -->
-  <!-- ===================================================== -->
-  <link name="caster_link">
-    <visual>
-      <origin xyz="0 0 0" rpy="0 0 0"/>
-      <geometry>
-        <sphere radius="0.04"/>
-      </geometry>
-      <material name="caster_gray">
-        <color rgba="0.3 0.3 0.3 1"/>
+    <dynamics damping="0.0" friction="0.0"/>
+  </joint>
+  <!-- ===================================================== -->
+  <!-- REAR LEFT WHEEL (driven, no steering)                  -->
+  <!-- ===================================================== -->
+  <link name="rear_left_wheel_link">
+    <visual>
+      <origin xyz="0 0 0" rpy="1.5708 0 0"/>
+      <geometry>
+        <cylinder radius="0.03" length="0.02"/>
+      </geometry>
+      <material name="black">
+        <color rgba="0.05 0.05 0.05 1"/>
       </material>
     </visual>
     <collision>
-      <origin xyz="0 0 0" rpy="0 0 0"/>
-      <geometry>
-        <sphere radius="0.04"/>
+      <origin xyz="0 0 0" rpy="1.5708 0 0"/>
+      <geometry>
+        <cylinder radius="0.03" length="0.02"/>
       </geometry>
     </collision>
     <inertial>
       <origin xyz="0 0 0" rpy="0 0 0"/>
-      <mass value="0.1"/>
-      <inertia
-        ixx="0.0001"
-        ixy="0.0"
-        ixz="0.0"
-        iyy="0.0001"
-        iyz="0.0"
-        izz="0.0001"/>
-    </inertial>
-  </link>
-  <joint name="caster_joint" type="fixed">
-    <parent link="base_link"/>
-    <child link="caster_link"/>
-    <!-- Fixed caster z-offset from -0.09 to -0.05 to prevent ground penetration -->
-    <origin
-      xyz="-0.14 0 -0.05"
-      rpy="0 0 0"/>
-  </joint>
-  <!-- ===================================================== -->
-  <!-- LIDAR                                                 -->
+      <mass value="0.15"/>
+      <inertia ixx="0.0001" ixy="0.0" ixz="0.0"
+                iyy="0.0001" iyz="0.0" izz="0.0001"/>
+    </inertial>
+  </link>
+  <joint name="rear_left_wheel_joint" type="continuous">
+    <parent link="base_link"/>
+    <child link="rear_left_wheel_link"/>
+    <origin xyz="-0.09 0.085 -0.03" rpy="0 0 0"/>
+    <axis xyz="0 1 0"/>
+    <dynamics damping="0.1" friction="0.1"/>
+  </joint>
+  <!-- ===================================================== -->
+  <!-- REAR RIGHT WHEEL (driven, no steering)                 -->
+  <!-- ===================================================== -->
+  <link name="rear_right_wheel_link">
+    <visual>
+      <origin xyz="0 0 0" rpy="1.5708 0 0"/>
+      <geometry>
+        <cylinder radius="0.03" length="0.02"/>
+      </geometry>
+      <material name="black">
+        <color rgba="0.05 0.05 0.05 1"/>
+      </material>
+    </visual>
+    <collision>
+      <origin xyz="0 0 0" rpy="1.5708 0 0"/>
+      <geometry>
+        <cylinder radius="0.03" length="0.02"/>
+      </geometry>
+    </collision>
+    <inertial>
+      <origin xyz="0 0 0" rpy="0 0 0"/>
+      <mass value="0.15"/>
+      <inertia ixx="0.0001" ixy="0.0" ixz="0.0"
+                iyy="0.0001" iyz="0.0" izz="0.0001"/>
+    </inertial>
+  </link>
+  <joint name="rear_right_wheel_joint" type="continuous">
+    <parent link="base_link"/>
+    <child link="rear_right_wheel_link"/>
+    <origin xyz="-0.09 -0.085 -0.02" rpy="0 0 0"/>
+    <axis xyz="0 1 0"/>
+    <dynamics damping="0.0" friction="0.0"/>
+  </joint>
+  <!-- ===================================================== -->
+  <!-- LIDAR (unchanged, mounting height fixed to new chassis) -->
   <!-- ===================================================== -->
   <link name="lidar_link">
@@ -180,7 +272,5 @@
       <origin xyz="0 0 0" rpy="0 0 0"/>
       <geometry>
-        <cylinder
-          radius="0.04"
-          length="0.03"/>
+        <cylinder radius="0.04" length="0.03"/>
       </geometry>
       <material name="lidar_black">
@@ -191,11 +281,6 @@
       <origin xyz="0 0 0" rpy="0 0 0"/>
       <mass value="0.05"/>
-      <inertia
-        ixx="0.0001"
-        ixy="0.0"
-        ixz="0.0"
-        iyy="0.0001"
-        iyz="0.0"
-        izz="0.0001"/>
+      <inertia ixx="0.0001" ixy="0.0" ixz="0.0"
+                iyy="0.0001" iyz="0.0" izz="0.0001"/>
     </inertial>
   </link>
@@ -203,17 +288,15 @@
     <parent link="base_link"/>
     <child link="lidar_link"/>
-    <origin
-      xyz="0 0 0.10"
-      rpy="0 0 0"/>
-  </joint>
-  <!-- ===================================================== -->
-  <!-- LIDAR GAZEBO SENSOR                                   -->
+    <!-- was 0.10 above a 0.15-tall chassis; adjusted for the
+         new 0.05-tall chassis so the lidar still clears the top -->
+    <origin xyz="0 0 0.05" rpy="0 0 0"/>
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