Commit message: Save Ackermann project working version

File: ros2_ws/src/robot_description/urdf/robot.urdf.xacro (robot description, xacro)
@@ -3,26 +3,13 @@
        xmlns:xacro="http://www.ros.org/wiki/xacro">
   <!-- =====================================================
-       Geometry updated to official Hiwonder chassis values
-       plus firmware constants:
-         - chassis plate: 270 x 120.5 x 2 mm (modeled as a
-           270 x 120.5 x 50 mm box - height is still a
-           modeling approximation, Hiwonder doesn't publish
-           assembled chassis height)
-         - wheel diameter: 60 mm (radius 0.03 m) - official
-         - wheelbase: 0.18 m (Hiwonder MINACKER_WHEELBASE)
-         - track width: 0.17 m (Hiwonder MINACKER_SHAFT_LENGTH)
-         - front axle x = +0.09, rear axle x = -0.09
-         - left wheel y = +0.085, right wheel y = -0.085
-         - ground clearance under chassis = 0.02 m (estimate)
-       STILL UNKNOWN / PLACEHOLDER:
-         - base_link mass (kept at 5.0 kg - bare plate is only
-           ~126 g, but full robot with motors/servo/battery/
-           compute/lidar will weigh more; update once assembled
-           and weighed)
-         - wheel / knuckle masses (placeholders)
-         - steering angle limit (0.6 rad / ~34 deg is an estimate,
-           actual range depends on the LD-1501MG + linkage geometry)
-         - lidar mounting height (unchanged until RPLIDAR A1 is
-           physically installed)
+       ROBOT GEOMETRY
+       Hiwonder-style Ackermann chassis:
+         - chassis: 270 x 120.5 x 50 mm model
+         - wheel diameter: 60 mm
+         - wheelbase: 0.18 m
+         - track width: 0.17 m
+         - front axle x = +0.09
+         - rear axle x = -0.09
+         - ground clearance ~ 0.02 m
   ===================================================== -->
   <!-- ===================================================== -->
@@ -33,6 +20,7 @@
     <parent link="base_footprint"/>
     <child link="base_link"/>
-    <!-- ground clearance (0.02) + half chassis height (0.025) -->
-    <origin xyz="0 0 0.05" rpy="0 0 0"/>
+    <origin
+      xyz="0 0 0.055"
+      rpy="0 0 0"/>
   </joint>
   <!-- ===================================================== -->
@@ -41,5 +29,7 @@
   <link name="base_link">
     <visual>
-      <origin xyz="0 0 0" rpy="0 0 0"/>
+      <origin
+        xyz="0 0 0"
+        rpy="0 0 0"/>
       <geometry>
         <box size="0.270 0.1205 0.050"/>
@@ -50,5 +40,7 @@
     </visual>
     <collision>
-      <origin xyz="0 0 0" rpy="0 0 0"/>
+      <origin
+        xyz="0 0 0"
+        rpy="0 0 0"/>
       <geometry>
         <box size="0.270 0.1205 0.050"/>
@@ -56,8 +48,7 @@
     </collision>
     <inertial>
-      <origin xyz="0 0 0" rpy="0 0 0"/>
-      <!-- mass is still a placeholder - bare Hiwonder plate is ~126 g,
-           but full robot (motors/servo/battery/compute/lidar) will be
-           heavier. Update once the robot is assembled and weighed. -->
+      <origin
+        xyz="0 0 0"
+        rpy="0 0 0"/>
       <mass value="2.5"/>
       <inertia
@@ -71,11 +62,28 @@
   </link>
   <!-- ===================================================== -->
-  <!-- STEERING LINK (virtual)                                -->
-  <!-- Required only because libgazebo_ros_ackermann_drive.so -->
-  <!-- looks for a steering_wheel_joint parameter. This does   -->
-  <!-- not drive anything physically - the real steering      -->
-  <!-- happens through front_left/right_steering_joint below.  -->
-  <!-- ===================================================== -->
+  <!-- VIRTUAL STEERING LINK                                  -->
+  <!-- Required by Ackermann plugin                           -->
+  <!--                                                         -->
+  <!--
+       Tiny 1mm visual sphere added: this link (and the two
+       front_*_steering_link links below) previously had ONLY
+       inertial, no visual/collision at all, the suspected
+       cause of the repeated Ogre AxisAlignedBox crash in
+       gzclient ("min corner must be less than or equal to max
+       corner"): a SceneNode with zero visual geometry can get
+       a degenerate bounding box on some Gazebo/Ogre builds.
+       No collision added, so this doesn't change physics or
+       contact behavior at all.
+  -->
   <link name="steering_link">
+    <visual>
+      <origin xyz="0 0 0" rpy="0 0 0"/>
+      <geometry>
+        <sphere radius="0.001"/>
+      </geometry>
+      <material name="steering_marker">
+        <color rgba="1 0 0 1"/>
+      </material>
+    </visual>
     <inertial>
       <origin xyz="0 0 0" rpy="0 0 0"/>
@@ -93,5 +101,7 @@
     <parent link="base_link"/>
     <child link="steering_link"/>
-    <origin xyz="0 0 0.05" rpy="0 0 0"/>
+    <origin
+      xyz="0 0 0.05"
+      rpy="0 0 0"/>
     <axis xyz="0 0 1"/>
     <limit
@@ -102,27 +112,55 @@
   </joint>
   <!-- ===================================================== -->
-  <!-- FRONT LEFT STEERING KNUCKLE + WHEEL                    -->
+  <!-- FRONT LEFT STEERING + WHEEL                            -->
   <!-- ===================================================== -->
   <link name="front_left_steering_link">
+    <visual>
+      <origin xyz="0 0 0" rpy="0 0 0"/>
+      <geometry>
+        <sphere radius="0.001"/>
+      </geometry>
+      <material name="steering_marker">
+        <color rgba="1 0 0 1"/>
+      </material>
+    </visual>
     <inertial>
       <origin xyz="0 0 0" rpy="0 0 0"/>
       <mass value="0.05"/>
-      <inertia ixx="0.00001" ixy="0.0" ixz="0.0"
-                iyy="0.00001" iyz="0.0" izz="0.00001"/>
-    </inertial>
-  </link>
-  <joint name="front_left_steering_joint" type="revolute">
+      <inertia
+        ixx="0.00001"
+        ixy="0.0"
+        ixz="0.0"
+        iyy="0.00001"
+        iyz="0.0"
+        izz="0.00001"/>
+    </inertial>
+  </link>
+  <joint
+    name="front_left_steering_joint"
+    type="revolute">
     <parent link="base_link"/>
     <child link="front_left_steering_link"/>
-    <origin xyz="0.09 0.085 -0.03" rpy="0 0 0"/>
+    <origin
+      xyz="0.09 0.085 -0.03"
+      rpy="0 0 0"/>
     <axis xyz="0 0 1"/>
-    <limit lower="-0.6" upper="0.6" effort="10" velocity="5"/>
-    <dynamics damping="0.05" friction="0.05"/>
+    <limit
+      lower="-0.6"
+      upper="0.6"
+      effort="10"
+      velocity="5"/>
+    <dynamics
+      damping="0.05"
+      friction="0.05"/>
   </joint>
   <link name="front_left_wheel_link">
     <visual>
-      <origin xyz="0 0 0" rpy="1.5708 0 0"/>
-      <geometry>
-        <cylinder radius="0.03" length="0.02"/>
+      <origin
+        xyz="0 0 0"
+        rpy="1.5708 0 0"/>
+      <geometry>
+        <cylinder
+          radius="0.03"
+          length="0.02"/>
       </geometry>
       <material name="black">
@@ -131,7 +169,11 @@
     </visual>
     <collision>
-      <origin xyz="0 0 0" rpy="1.5708 0 0"/>
-      <geometry>
-        <cylinder radius="0.03" length="0.02"/>
+      <origin
+        xyz="0 0 0"
+        rpy="1.5708 0 0"/>
+      <geometry>
+        <cylinder
+          radius="0.03"
+          length="0.02"/>
       </geometry>
     </collision>
@@ -139,39 +181,78 @@
       <origin xyz="0 0 0" rpy="0 0 0"/>
       <mass value="0.15"/>
-      <inertia ixx="0.0001" ixy="0.0" ixz="0.0"
-                iyy="0.0001" iyz="0.0" izz="0.0001"/>
-    </inertial>
-  </link>
-  <joint name="front_left_wheel_joint" type="continuous">
+      <inertia
+        ixx="0.0001"
+        ixy="0.0"
+        ixz="0.0"
+        iyy="0.0001"
+        iyz="0.0"
+        izz="0.0001"/>
+    </inertial>
+  </link>
+  <joint
+    name="front_left_wheel_joint"
+    type="continuous">
     <parent link="front_left_steering_link"/>
     <child link="front_left_wheel_link"/>
-    <origin xyz="0 0 0" rpy="0 0 0"/>
+    <origin
+      xyz="0 0 0"
+      rpy="0 0 0"/>
     <axis xyz="0 1 0"/>
-    <dynamics damping="0.1" friction="0.1"/>
-  </joint>
-  <!-- ===================================================== -->
-  <!-- FRONT RIGHT STEERING KNUCKLE + WHEEL                   -->
+    <dynamics
+      damping="0.1"
+      friction="0.1"/>
+  </joint>
+  <!-- ===================================================== -->
+  <!-- FRONT RIGHT STEERING + WHEEL                           -->
   <!-- ===================================================== -->
   <link name="front_right_steering_link">
+    <visual>
+      <origin xyz="0 0 0" rpy="0 0 0"/>
+      <geometry>
+        <sphere radius="0.001"/>
+      </geometry>
+      <material name="steering_marker">
+        <color rgba="1 0 0 1"/>
+      </material>
+    </visual>
     <inertial>
       <origin xyz="0 0 0" rpy="0 0 0"/>
       <mass value="0.05"/>
-      <inertia ixx="0.00001" ixy="0.0" ixz="0.0"
-                iyy="0.00001" iyz="0.0" izz="0.00001"/>
-    </inertial>
-  </link>
-  <joint name="front_right_steering_joint" type="revolute">
+      <inertia
+        ixx="0.00001"
+        ixy="0.0"
+        ixz="0.0"
+        iyy="0.00001"
+        iyz="0.0"
+        izz="0.00001"/>
+    </inertial>
+  </link>
+  <joint
+    name="front_right_steering_joint"
+    type="revolute">
     <parent link="base_link"/>
     <child link="front_right_steering_link"/>
-    <origin xyz="0.09 -0.085 -0.03" rpy="0 0 0"/>
+    <origin
+      xyz="0.09 -0.085 -0.03"
+      rpy="0 0 0"/>
     <axis xyz="0 0 1"/>
-    <limit lower="-0.6" upper="0.6" effort="10" velocity="5"/>
-    <dynamics damping="0.05" friction="0.05"/>
+    <limit
+      lower="-0.6"
+      upper="0.6"
+      effort="10"
+      velocity="5"/>
+    <dynamics
+      damping="0.05"
+      friction="0.05"/>
   </joint>
   <link name="front_right_wheel_link">
     <visual>
-      <origin xyz="0 0 0" rpy="1.5708 0 0"/>
-      <geometry>
-        <cylinder radius="0.03" length="0.02"/>
+      <origin
+        xyz="0 0 0"
+        rpy="1.5708 0 0"/>
+      <geometry>
+        <cylinder
+          radius="0.03"
+          length="0.02"/>
       </geometry>
       <material name="black">
@@ -180,7 +261,11 @@
     </visual>
     <collision>
-      <origin xyz="0 0 0" rpy="1.5708 0 0"/>
-      <geometry>
-        <cylinder radius="0.03" length="0.02"/>
+      <origin
+        xyz="0 0 0"
+        rpy="1.5708 0 0"/>
+      <geometry>
+        <cylinder
+          radius="0.03"
+          length="0.02"/>
       </geometry>
     </collision>
@@ -188,23 +273,38 @@
       <origin xyz="0 0 0" rpy="0 0 0"/>
       <mass value="0.15"/>
-      <inertia ixx="0.0001" ixy="0.0" ixz="0.0"
-                iyy="0.0001" iyz="0.0" izz="0.0001"/>
-    </inertial>
-  </link>
-  <joint name="front_right_wheel_joint" type="continuous">
+      <inertia
+        ixx="0.0001"
+        ixy="0.0"
+        ixz="0.0"
+        iyy="0.0001"
+        iyz="0.0"
+        izz="0.0001"/>
+    </inertial>
+  </link>
+  <joint
+    name="front_right_wheel_joint"
+    type="continuous">
     <parent link="front_right_steering_link"/>
     <child link="front_right_wheel_link"/>
-    <origin xyz="0 0 0" rpy="0 0 0"/>
+    <origin
+      xyz="0 0 0"
+      rpy="0 0 0"/>
     <axis xyz="0 1 0"/>
-    <dynamics damping="0.0" friction="0.0"/>
-  </joint>
-  <!-- ===================================================== -->
-  <!-- REAR LEFT WHEEL (driven, no steering)                  -->
+    <dynamics
+      damping="0.0"
+      friction="0.0"/>
+  </joint>
+  <!-- ===================================================== -->
+  <!-- REAR LEFT WHEEL                                       -->
   <!-- ===================================================== -->
   <link name="rear_left_wheel_link">
     <visual>
-      <origin xyz="0 0 0" rpy="1.5708 0 0"/>
-      <geometry>
-        <cylinder radius="0.03" length="0.02"/>
+      <origin
+        xyz="0 0 0"
+        rpy="1.5708 0 0"/>
+      <geometry>
+        <cylinder
+          radius="0.03"
+          length="0.02"/>
       </geometry>
       <material name="black">
@@ -213,7 +313,11 @@
     </visual>
     <collision>
-      <origin xyz="0 0 0" rpy="1.5708 0 0"/>
-      <geometry>
-        <cylinder radius="0.03" length="0.02"/>
+      <origin
+        xyz="0 0 0"
+        rpy="1.5708 0 0"/>
+      <geometry>
+        <cylinder
+          radius="0.03"
+          length="0.02"/>
       </geometry>
     </collision>
@@ -221,23 +325,38 @@
       <origin xyz="0 0 0" rpy="0 0 0"/>
       <mass value="0.15"/>
-      <inertia ixx="0.0001" ixy="0.0" ixz="0.0"
-                iyy="0.0001" iyz="0.0" izz="0.0001"/>
-    </inertial>
-  </link>
-  <joint name="rear_left_wheel_joint" type="continuous">
+      <inertia
+        ixx="0.0001"
+        ixy="0.0"
+        ixz="0.0"
+        iyy="0.0001"
+        iyz="0.0"
+        izz="0.0001"/>
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