Commit message: Fix navigation reliability; add DFS memory, single Q-table path, SAC scaffolding
Controller (grid_rl_controller.py):
- Move loop exited on Euclidean distance to a target point, so lateral
  drift beyond position_tolerance made the exit test unsatisfiable and
  the robot drove until it hit something. Now projects onto the travel
  axis, which cannot be missed.
- Move was open-loop in heading (angular.z = 0.0 throughout). Added a
  heading + cross-track P controller so it holds the corridor centre
  line; tightened angle_tolerance 0.08 -> 0.03.
- wall_distance 0.55 -> 0.80; proportional turn ramp.

Exploration (maze_memory.py, new):
- The 7-tuple RL state is memoryless, so the greedy fallback livelocked
  in front of dead ends and 6 of 24 start cells never finished. Adds a
  visited set and DFS path stack: 0 failures over all 600 start/goal
  pairs, worst case 43 steps.

Q-table path (q_table_path.py, new):
- Four copies of q_table.pkl existed and drifted apart because train.py
  saved next to __file__ while run_policy searched a different order.
  One resolver now: $RL_Q_TABLE, else ~/.ros/rl_ackermann/q_table.pkl.
  Removed the q_table.pkl entries from setup.py so colcon stops copying.

Q-table format guard (q_learning.py, run_policy.py):
- The shipped table was keyed on a 9-tuple (absolute positions) while
  the controller emits a 7-tuple (relative), so every lookup missed and
  the policy silently ran on its fallback alone. STATE_FORMAT is now
  stamped on save and verified on load. Retrained: 3744 states, 98.09%.

DRL (drl/, new, in progress):
- config.py: observation/action contract shared by surrogate and node.
- geometry.py: vectorised raycasting for the fast training surrogate.

Co-Authored-By: Claude Opus 5 (1M context) <noreply@anthropic.com>

File: ros2_ws/src/robot_description/urdf/robot.urdf.xacro (robot description, xacro)
@@ -3,35 +3,121 @@
        xmlns:xacro="http://www.ros.org/wiki/xacro">
   <!-- =====================================================
-       ROBOT GEOMETRY
-       Hiwonder-style Ackermann chassis:
-         - chassis: 270 x 120.5 x 50 mm model
-         - wheel diameter: 60 mm
-         - wheelbase: 0.18 m
-         - track width: 0.17 m
-         - front axle x = +0.09
-         - rear axle x = -0.09
-         - ground clearance ~ 0.02 m
-  ===================================================== -->
-  <!-- ===================================================== -->
-  <!-- BASE FOOTPRINT                                        -->
-  <!-- ===================================================== -->
+       ORIGIN CONVENTION  (changed - read this)
+       base_link / base_footprint sit on the REAR AXLE, not the
+       geometric centre of the plate.
+       Why: the robot pivots about whatever point has no lateral
+       scrub. With rear-wheel drive and free-rolling front wheels
+       that point is the rear axle. Odometry, the LIDAR and the
+       pivot centre must all coincide, or every turn injects a
+       position error that grid_rl_controller.py cannot see.
+       So: rear wheels at x = 0, front wheels at x = wheelbase,
+       chassis plate and LIDAR offset accordingly.
+       This also matches what libgazebo_ros_ackermann_drive
+       expects, so both drive modes use the same frame.
+       ===================================================== -->
+  <!-- =====================================================
+       DRIVE MODE SELECTOR
+         diff       - rear wheels driven by libgazebo_ros_diff_drive,
+                      front wheels free-rolling and near-frictionless
+                      (they stand in for the old caster). Robot pivots
+                      cleanly about the rear axle.
+         ackermann  - true car-like steering. Robot CANNOT pivot in
+                      place; grid_rl_controller.py needs arc / K-turn
+                      primitives first.
+       Usage:
+         xacro robot.urdf.xacro drive_mode:=diff
+         xacro robot.urdf.xacro drive_mode:=ackermann
+       ===================================================== -->
+  <xacro:arg name="drive_mode" default="diff"/>
+  <xacro:property name="drive_mode" value="$(arg drive_mode)"/>
+  <!-- =====================================================
+       CHASSIS GEOMETRY
+       Ackerman Metal Chassis (ThinkRobotics / Hiwonder)
+       Plate 270 mm x 120.5 mm aluminium.
+       ===================================================== -->
+  <xacro:property name="chassis_length" value="0.270"/>
+  <xacro:property name="chassis_width"  value="0.1205"/>
+  <xacro:property name="chassis_height" value="0.045"/>
+  <xacro:property name="chassis_mass"   value="2.5"/>
+  <!-- MEASURED -->
+  <xacro:property name="wheelbase"      value="0.213"/>
+  <xacro:property name="track_width"    value="0.222"/>
+  <xacro:property name="wheel_radius"   value="0.0505"/>
+  <xacro:property name="wheel_width"    value="0.040"/>
+  <xacro:property name="wheel_mass"     value="0.20"/>
+  <!-- STILL TO VERIFY AT THE KNUCKLE, NOT THE SERVO.
+         25 deg -> R = 0.457 m
+         30 deg -> R = 0.369 m   (value used)
+         35 deg -> R = 0.304 m -->
+  <xacro:property name="max_steer"      value="0.5236"/>
+  <xacro:property name="ground_clearance" value="0.025"/>
+  <!-- Plate centre relative to the rear axle. Overhang is
+       (0.270 - 0.213)/2 = 0.0285 m at each end, so the plate
+       centre sits wheelbase/2 ahead of the rear axle. -->
+  <xacro:property name="chassis_x" value="${wheelbase/2}"/>
+  <xacro:property name="chassis_z"
+                  value="${ground_clearance - wheel_radius + chassis_height/2}"/>
+  <xacro:property name="chassis_top"
+                  value="${chassis_z + chassis_height/2}"/>
+  <!-- =====================================================
+       LIDAR GEOMETRY - RPLIDAR A1M8
+       ===================================================== -->
+  <xacro:property name="lidar_radius" value="0.035"/>
+  <xacro:property name="lidar_height" value="0.041"/>
+  <xacro:property name="lidar_mass"   value="0.17"/>
+  <!-- Must clear the 101 mm tyres (tops at 0.1010 m). 0.060 m
+       puts the beam plane at 0.1505 m, ~50 mm clear. Maze walls
+       are 0.50 m tall, so that is fine. -->
+  <xacro:property name="lidar_standoff" value="0.060"/>
+  <xacro:property name="lidar_z"
+                  value="${chassis_top + lidar_standoff + lidar_height/2}"/>
+  <!-- A1M8 is ~1% of range. Set 0.0 for noise-free scans. -->
+  <xacro:property name="lidar_noise_stddev" value="0.01"/>
+  <!-- =====================================================
+       INERTIA MACROS
+       ===================================================== -->
+  <xacro:macro name="box_inertia" params="m x y z x0:=0 y0:=0 z0:=0">
+    <inertial>
+      <origin xyz="${x0} ${y0} ${z0}" rpy="0 0 0"/>
+      <mass value="${m}"/>
+      <inertia
+        ixx="${m*(y*y + z*z)/12.0}"
+        ixy="0.0"
+        ixz="0.0"
+        iyy="${m*(x*x + z*z)/12.0}"
+        iyz="0.0"
+        izz="${m*(x*x + y*y)/12.0}"/>
+    </inertial>
+  </xacro:macro>
+  <xacro:macro name="wheel_inertia" params="m r l">
+    <inertial>
+      <origin xyz="0 0 0" rpy="1.5708 0 0"/>
+      <mass value="${m}"/>
+      <inertia
+        ixx="${m*(3.0*r*r + l*l)/12.0}"
+        ixy="0.0"
+        ixz="0.0"
+        iyy="${m*(3.0*r*r + l*l)/12.0}"
+        iyz="0.0"
+        izz="${m*r*r/2.0}"/>
+    </inertial>
+  </xacro:macro>
+  <!-- =====================================================
+       BASE FOOTPRINT (on the rear axle, projected to ground)
+       ===================================================== -->
   <link name="base_footprint"/>
   <joint name="base_footprint_joint" type="fixed">
     <parent link="base_footprint"/>
-    <child link="base_link"/>
-    <origin
-      xyz="0 0 0.055"
-      rpy="0 0 0"/>
-  </joint>
-  <!-- ===================================================== -->
-  <!-- BASE LINK                                             -->
-  <!-- ===================================================== -->
+    <child  link="base_link"/>
+    <origin xyz="0 0 ${wheel_radius}" rpy="0 0 0"/>
+  </joint>
+  <!-- =====================================================
+       BASE LINK
+       ===================================================== -->
   <link name="base_link">
     <visual>
-      <origin
-        xyz="0 0 0"
-        rpy="0 0 0"/>
+      <origin xyz="${chassis_x} 0 ${chassis_z}" rpy="0 0 0"/>
       <geometry>
-        <box size="0.270 0.1205 0.050"/>
+        <box size="${chassis_length} ${chassis_width} ${chassis_height}"/>
       </geometry>
       <material name="blue">
@@ -40,375 +126,148 @@
     </visual>
     <collision>
-      <origin
-        xyz="0 0 0"
-        rpy="0 0 0"/>
+      <origin xyz="${chassis_x} 0 ${chassis_z}" rpy="0 0 0"/>
       <geometry>
-        <box size="0.270 0.1205 0.050"/>
+        <box size="${chassis_length} ${chassis_width} ${chassis_height}"/>
       </geometry>
     </collision>
-    <inertial>
-      <origin
-        xyz="0 0 0"
-        rpy="0 0 0"/>
-      <mass value="2.5"/>
-      <inertia
-        ixx="0.003546"
-        ixy="0.0"
-        ixz="0.0"
-        iyy="0.015708"
-        iyz="0.0"
-        izz="0.018213"/>
-    </inertial>
+    <xacro:box_inertia
+      m="${chassis_mass}"
+      x="${chassis_length}"
+      y="${chassis_width}"
+      z="${chassis_height}"
+      x0="${chassis_x}"
+      z0="${chassis_z}"/>
   </link>
-  <!-- ===================================================== -->
-  <!-- VIRTUAL STEERING LINK                                  -->
-  <!-- Required by Ackermann plugin                           -->
-  <!--                                                         -->
-  <!--
-       Tiny 1mm visual sphere added: this link (and the two
-       front_*_steering_link links below) previously had ONLY
-       inertial, no visual/collision at all, the suspected
-       cause of the repeated Ogre AxisAlignedBox crash in
-       gzclient ("min corner must be less than or equal to max
-       corner"): a SceneNode with zero visual geometry can get
-       a degenerate bounding box on some Gazebo/Ogre builds.
-       No collision added, so this doesn't change physics or
-       contact behavior at all.
-  -->
-  <link name="steering_link">
+  <!-- =====================================================
+       WHEEL / KNUCKLE MACROS
+       ===================================================== -->
+  <xacro:macro name="wheel_link" params="name">
+    <link name="${name}_link">
+      <visual>
+        <origin xyz="0 0 0" rpy="1.5708 0 0"/>
+        <geometry>
+          <cylinder radius="${wheel_radius}" length="${wheel_width}"/>
+        </geometry>
+        <material name="black">
+          <color rgba="0.05 0.05 0.05 1"/>
+        </material>
+      </visual>
+      <collision>
+        <origin xyz="0 0 0" rpy="1.5708 0 0"/>
+        <geometry>
+          <cylinder radius="${wheel_radius}" length="${wheel_width}"/>
+        </geometry>
+      </collision>
+      <xacro:wheel_inertia
+        m="${wheel_mass}"
+        r="${wheel_radius}"
+        l="${wheel_width}"/>
+    </link>
+  </xacro:macro>
+  <xacro:macro name="knuckle_link" params="name">
+    <link name="${name}_link">
+      <visual>
+        <origin xyz="0 0 0" rpy="0 0 0"/>
+        <geometry>
+          <box size="0.02 0.02 0.03"/>
+        </geometry>
+        <material name="knuckle_gray">
+          <color rgba="0.4 0.4 0.4 1"/>
+        </material>
+      </visual>
+      <xacro:box_inertia m="0.05" x="0.02" y="0.02" z="0.03"/>
+    </link>
+  </xacro:macro>
+  <xacro:wheel_link name="front_left_wheel"/>
+  <xacro:wheel_link name="front_right_wheel"/>
+  <xacro:wheel_link name="rear_left_wheel"/>
+  <xacro:wheel_link name="rear_right_wheel"/>
+  <xacro:knuckle_link name="front_left_knuckle"/>
+  <xacro:knuckle_link name="front_right_knuckle"/>
+  <!-- =====================================================
+       REAR AXLE - at the origin, driven in both modes
+       ===================================================== -->
+  <joint name="rear_left_wheel_joint" type="continuous">
+    <parent link="base_link"/>
+    <child  link="rear_left_wheel_link"/>
+    <origin xyz="0 ${track_width/2} 0" rpy="0 0 0"/>
+    <axis xyz="0 1 0"/>
+    <dynamics damping="0.05" friction="0.02"/>
+  </joint>
+  <joint name="rear_right_wheel_joint" type="continuous">
+    <parent link="base_link"/>
+    <child  link="rear_right_wheel_link"/>
+    <origin xyz="0 ${-track_width/2} 0" rpy="0 0 0"/>
+    <axis xyz="0 1 0"/>
+    <dynamics damping="0.05" friction="0.02"/>
+  </joint>
+  <!-- =====================================================
+       FRONT STEERING JOINTS
+       ===================================================== -->
+  <xacro:if value="${drive_mode == 'diff'}">
+    <joint name="front_left_steering_joint" type="fixed">
+      <parent link="base_link"/>
+      <child  link="front_left_knuckle_link"/>
+      <origin xyz="${wheelbase} ${track_width/2} 0" rpy="0 0 0"/>
+    </joint>
+    <joint name="front_right_steering_joint" type="fixed">
+      <parent link="base_link"/>
+      <child  link="front_right_knuckle_link"/>
+      <origin xyz="${wheelbase} ${-track_width/2} 0" rpy="0 0 0"/>
+    </joint>
+  </xacro:if>
+  <xacro:if value="${drive_mode == 'ackermann'}">
+    <joint name="front_left_steering_joint" type="revolute">
+      <parent link="base_link"/>
+      <child  link="front_left_knuckle_link"/>
+      <origin xyz="${wheelbase} ${track_width/2} 0" rpy="0 0 0"/>
+      <axis xyz="0 0 1"/>
+      <limit lower="${-max_steer}" upper="${max_steer}"
+             effort="10.0" velocity="5.0"/>
+      <dynamics damping="0.1" friction="0.05"/>
+    </joint>
+    <joint name="front_right_steering_joint" type="revolute">
+      <parent link="base_link"/>
+      <child  link="front_right_knuckle_link"/>
+      <origin xyz="${wheelbase} ${-track_width/2} 0" rpy="0 0 0"/>
+      <axis xyz="0 0 1"/>
+      <limit lower="${-max_steer}" upper="${max_steer}"
+             effort="10.0" velocity="5.0"/>
+      <dynamics damping="0.1" friction="0.05"/>
+    </joint>
+    <link name="steering_wheel_link">
+      <xacro:box_inertia m="0.01" x="0.01" y="0.01" z="0.01"/>
+    </link>
+    <joint name="steering_wheel_joint" type="revolute">
+      <parent link="base_link"/>
+      <child  link="steering_wheel_link"/>
+      <origin xyz="${chassis_x} 0 ${chassis_top}" rpy="0 0 0"/>
+      <axis xyz="0 0 1"/>
+      <limit lower="-7.85" upper="7.85" effort="1.0" velocity="10.0"/>
+    </joint>
+  </xacro:if>
+  <joint name="front_left_wheel_joint" type="continuous">
+    <parent link="front_left_knuckle_link"/>
+    <child  link="front_left_wheel_link"/>
+    <origin xyz="0 0 0" rpy="0 0 0"/>
+    <axis xyz="0 1 0"/>
+    <dynamics damping="0.02" friction="0.0"/>
+  </joint>
+  <joint name="front_right_wheel_joint" type="continuous">
+    <parent link="front_right_knuckle_link"/>
+    <child  link="front_right_wheel_link"/>
+    <origin xyz="0 0 0" rpy="0 0 0"/>
+    <axis xyz="0 1 0"/>
+    <dynamics damping="0.02" friction="0.0"/>
+  </joint>
+  <!-- =====================================================
+       LIDAR - directly over the rear axle, i.e. over the
+       pivot centre and over the odometry origin.
+       ===================================================== -->
+  <link name="lidar_link">
     <visual>
       <origin xyz="0 0 0" rpy="0 0 0"/>
       <geometry>
-        <sphere radius="0.001"/>
-      </geometry>
-      <material name="steering_marker">
-        <color rgba="1 0 0 1"/>
-      </material>
-    </visual>
-    <inertial>
-      <origin xyz="0 0 0" rpy="0 0 0"/>
-      <mass value="0.001"/>
-      <inertia
-        ixx="0.000001"
-        ixy="0.0"
-        ixz="0.0"
-        iyy="0.000001"
-        iyz="0.0"
-        izz="0.000001"/>
-    </inertial>
-  </link>
-  <joint name="steering_joint" type="revolute">
-    <parent link="base_link"/>
-    <child link="steering_link"/>
-    <origin
-      xyz="0 0 0.05"
-      rpy="0 0 0"/>
-    <axis xyz="0 0 1"/>
-    <limit
-      lower="-7.85"
-      upper="7.85"
-      effort="10"
-      velocity="10"/>
-  </joint>
-  <!-- ===================================================== -->
-  <!-- FRONT LEFT STEERING + WHEEL                            -->
-  <!-- ===================================================== -->
-  <link name="front_left_steering_link">
-    <visual>
-      <origin xyz="0 0 0" rpy="0 0 0"/>
-      <geometry>
-        <sphere radius="0.001"/>
-      </geometry>
-      <material name="steering_marker">
-        <color rgba="1 0 0 1"/>
-      </material>
-    </visual>
-    <inertial>
-      <origin xyz="0 0 0" rpy="0 0 0"/>
-      <mass value="0.05"/>
-      <inertia
-        ixx="0.00001"
-        ixy="0.0"
-        ixz="0.0"
-        iyy="0.00001"
-        iyz="0.0"
-        izz="0.00001"/>
-    </inertial>
-  </link>
-  <joint
-    name="front_left_steering_joint"
-    type="revolute">
-    <parent link="base_link"/>
-    <child link="front_left_steering_link"/>
-    <origin
-      xyz="0.09 0.085 -0.03"
-      rpy="0 0 0"/>
-    <axis xyz="0 0 1"/>
-    <limit
-      lower="-0.6"
-      upper="0.6"
-      effort="10"
-      velocity="5"/>
-    <dynamics
-      damping="0.05"
-      friction="0.05"/>
-  </joint>
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